Commit message: Tf changes

File: src/visiondrone/rviz/drone.urdf (robot description, URDF)
Before this commit: robot drone, 1 links, 0 joints
Links:
- link base_link: geometry visual mesh filename=package://visiondrone/rviz/drone.stl scale=0.001 0.001 0.001

Commit message: Cleanup, we no longer depend on robot_localization

File: src/visiondrone/rviz/drone.urdf (robot description, URDF)
Before this commit: robot drone, 1 links, 0 joints
Links:
- link base_link: geometry visual mesh filename=package://visiondrone/rviz/drone.stl scale=0.01 0.01 0.01
